File: linear_supply.kicad_pcb (KiCad board)
At the start: 2 copper layers, 96.5 x 94 mm, 21 parts, among them J2 Conn_01x02_Socket, Q1 BD139, Q2 TIP31C, Q3 2N2222, T1 Transformer_1P_1S, U1 OP07, j1 Conn_01x02_Socket

Commit message: i uploded this here
Routing:
- net Net-(D3-+): track 117.5 -> 124.2 mm
- net Net-(U1--): track 31.0 -> 27.8 mm
- net Net-(T1-SA): track 40.2 -> 41.9 mm
- net Net-(J2-Pin_1): track 95.7 -> 94.2 mm
Changed lines of the file:
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@@
 	)
 	(setup
+		(stackup
+			(layer "F.SilkS"
+				(type "Top Silk Screen")
+			)
+			(layer "F.Paste"
+				(type "Top Solder Paste")
+			)
+			(layer "F.Mask"
+				(type "Top Solder Mask")
+				(thickness 0.01)
+			)
+			(layer "F.Cu"
+				(type "copper")
+				(thickness 0.035)
+			)
+			(layer "dielectric 1"
+				(type "core")
+				(thickness 1.51)
+				(material "FR4")
+				(epsilon_r 4.5)
+				(loss_tangent 0.02)
+			)
+			(layer "B.Cu"
+				(type "copper")
+				(thickness 0.035)
+			)
+			(layer "B.Mask"
+				(type "Bottom Solder Mask")
+				(thickness 0.01)
+			)
+			(layer "B.Paste"
+				(type "Bottom Solder Paste")
+			)
+			(layer "B.SilkS"
+				(type "Bottom Silk Screen")
+			)
+			(copper_finish "None")
+			(dielectric_constraints no)
+		)
 		(pad_to_mask_clearance 0)
 		(allow_soldermask_bridges_in_footprints no)
@@
 	)
 	(segment
-		(start 185.155354 60.729646)
-		(end 177.5725 68.3125)
-		(width 1.4)
-		(layer "F.Cu")
-		(net 2)
-	)
-	(segment
 		(start 182.92 73.66)
 		(end 182.92 81.3)
@@
 	)
 	(segment
+		(start 182.92 62.965)
+		(end 185.155354 60.729646)
+		(width 1.4)
+		(layer "F.Cu")
+		(net 2)
+	)
+	(segment
 		(start 195.58 55.88)
 		(end 197.18 54.28)
@@
 	)
 	(segment
+		(start 182.92 73.66)
+		(end 182.92 62.965)
+		(width 1.4)
+		(layer "F.Cu")
+		(net 2)
+	)
+	(segment
 		(start 185.155354 55.88)
 		(end 195.58 55.88)
@@
 	)
 	(segment
-		(start 184.925025 106.185025)
-		(end 182.88 104.14)
-		(width 0.5)
+		(start 182.88 105.053654)
+		(end 184.506346 106.68)
+		(width 1.4)
 		(layer "B.Cu")
 		(net 2)
 	)
 	(segment
-		(start 193.04 119.38)
-		(end 193.04 119.6925)
-		(width 0.5)
+		(start 197.4325 121.28)
+		(end 197.4325 116.1525)
+		(width 1.4)
 		(layer "B.Cu")
 		(net 2)
 	)
 	(segment
-		(start 194.1775 120.83)
-		(end 196.9825 120.83)
-		(width 0.5)
+		(start 193.275 121.92)
+		(end 196.7925 121.92)
+		(width 1.4)
 		(layer "B.Cu")
 		(net 2)
 	)
 	(segment
-		(start 193.04 119.6925)
-		(end 194.1775 120.83)
-		(width 0.5)
+		(start 184.506346 106.68)
+		(end 187.96 106.68)
+		(width 1.4)
 		(layer "B.Cu")
 		(net 2)
 	)
 	(segment
-		(start 196.9825 115.7025)
-		(end 187.465025 106.185025)
-		(width 0.5)
+		(start 193.04 119.38)
+		(end 193.04 121.685)
+		(width 1.4)
 		(layer "B.Cu")
 		(net 2)
 	)
 	(segment
-		(start 187.465025 106.185025)
-		(end 184.925025 106.185025)
-		(width 0.5)
+		(start 187.96 106.68)
+		(end 197.4325 116.1525)
+		(width 1.4)
 		(layer "B.Cu")
 		(net 2)
 	)
 	(segment
-		(start 196.9825 120.83)
-		(end 196.9825 115.7025)
-		(width 0.5)
+		(start 196.7925 121.92)
+		(end 197.4325 121.28)
+		(width 1.4)
+		(layer "B.Cu")
+		(net 2)
+	)
+	(segment
+		(start 182.88 104.14)
+		(end 182.88 105.053654)
+		(width 1.4)
+		(layer "B.Cu")
+		(net 2)
+	)
+	(segment
+		(start 193.04 121.685)
+		(end 193.275 121.92)
+		(width 1.4)
 		(layer "B.Cu")
 		(net 2)
@@
 	)
 	(segment
-		(start 198.12 96.52)
-		(end 208.28 96.52)
+		(start 197.38 96.52)
+		(end 187.96 105.94)
 		(width 1.4)
 		(layer "F.Cu")
@@
 	)
 	(segment
-		(start 166.9 105.94)
-		(end 188.7 105.94)
+		(start 187.96 105.94)
+		(end 166.9 105.94)
 		(width 1.4)
 		(layer "F.Cu")
@@
 	)
 	(segment
+		(start 197.38 96.52)
+		(end 203.12 96.52)
+		(width 1.4)
+		(layer "F.Cu")
+		(net 3)
+	)
+	(segment
 		(start 208.015354 114.3)
 		(end 210.68 111.635354)
@@
 	)
 	(segment
-		(start 188.7 105.94)
-		(end 198.12 96.52)
+		(start 203.12 96.52)
+		(end 205.7 93.94)
 		(width 1.4)
 		(layer "F.Cu")
@@
 	)
 	(segment
-		(start 141.3975 84.585)
-		(end 150.97 75.0125)
-		(width 1.4)
+		(start 141.0975 108.11)
+		(end 141.0975 82.4225)
+		(width 2)
 		(layer "F.Cu")
 		(net 5)
 	)
 	(segment
-		(start 141.3975 108.41)
-		(end 141.3975 84.585)
-		(width 1.4)
+		(start 141.0975 82.4225)
+		(end 148.5075 75.0125)
+		(width 2)
+		(layer "F.Cu")
+		(net 5)
+	)
+	(segment
+		(start 148.5075 75.0125)
+		(end 150.97 75.0125)
+		(width 2)
 		(layer "F.Cu")
 		(net 5)
@@
 	(segment
 		(start 143.3975 110.41)
-		(end 141.3975 108.41)
-		(width 1.4)
+		(end 141.0975 108.11)
+		(width 2)
 		(layer "F.Cu")
 		(net 5)
 	)
 	(segment
-		(start 158.0975 67.885)
+		(start 161.25125 100.29125)
+		(end 161.25125 64.73125)
+		(width 2)
+		(layer "F.Cu")
+		(net 6)
+	)
+	(segment
+		(start 161.25125 64.73125)
 		(end 169.07 56.9125)
-		(width 1.4)
+		(width 2)
 		(layer "F.Cu")
 		(net 6)
 	)
 	(segment
-		(start 158.0975 108.41)
-		(end 158.0975 67.885)
-		(width 1.4)
+		(start 161.25125 100.29125)
+		(end 156.0975 105.445)
+		(width 2)
 		(layer "F.Cu")
 		(net 6)
 	)
 	(segment
-		(start 156.0975 110.41)
-		(end 158.0975 108.41)
-		(width 1.4)
+		(start 156.0975 105.445)
+		(end 156.0975 110.41)
+		(width 2)
 		(layer "F.Cu")
 		(net 6)
@@
 	(segment
 		(start 146.90132 85.02)
-		(end 144.78 85.02)
-		(width 1.4)
+		(end 156.0975 94.21618)
+		(width 2)
 		(layer "F.Cu")
 		(net 7)
@@
 	(segment
 		(start 156.0975 94.21618)
-		(end 146.90132 85.02)
-		(width 1.4)
+		(end 156.0975 100.41)
+		(width 2)
 		(layer "F.Cu")
 		(net 7)
 	)
 	(segment
-		(start 156.0975 100.41)
-		(end 156.0975 94.21618)
-		(width 1.4)
+		(start 144.78 85.02)
+		(end 146.90132 85.02)
+		(width 2)
 		(layer "F.Cu")
 		(net 7)
@@
 		(start 144.78 88.9)
 		(end 144.78 99.0275)
-		(width 1.4)
+		(width 2)
 		(layer "F.Cu")
 		(net 8)
@@
 		(start 144.78 99.0275)
 		(end 143.3975 100.41)
-		(width 1.4)
+		(width 2)
 		(layer "F.Cu")
 		(net 8)
@@
 	)
 	(segment
-		(start 177.8 86.36)
+		(start 170.18 88.9)
 		(end 170.18 93.98)
 		(width 0.5)
@@
 	)
 	(segment
-		(start 184.16 90.16)
-		(end 180.36 86.36)
-		(width 0.5)
-		(layer "B.Cu")
-		(net 14)
-	)
-	(segment
-		(start 170.18 88.9)
-		(end 170.18 93.98)
+		(start 165.1 83.82)
+		(end 170.18 88.9)
 		(width 0.5)
 		(layer "B.Cu")
@@
 	)
 	(segment
-		(start 180.36 86.36)
-		(end 177.8 86.36)
+		(start 184.16 90.16)
+		(end 180.34 93.98)
 		(width 0.5)
 		(layer "B.Cu")
@@
 	)
 	(segment
-		(start 165.1 83.82)
-		(end 170.18 88.9)
+		(start 180.34 93.98)
+		(end 170.18 93.98)
 		(width 0.5)
 		(layer "B.Cu")
